File: adsr7555_kassutronics.kicad_pcb (KiCad board)
At the start: 2 copper layers, 68.6 x 104.1 mm, 47 parts, among them J1 Power, J2 GateIn, J5 Atn Out, J6 Output, Q1 3904, Q2 3904, Q3 3904, Q4 3904, SW1 SW_Push, U1 7555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

Commit message: update PCB wiring worked on lower right
Parts:
- C3: footprint Capacitor_THT:CP_Radial_D4.0mm_P2.00mm -> Capacitor_THT:CP_Radial_D5.0mm_P2.50mm
Routing:
- net Net-(U2C-+): track 200.7 -> 195.6 mm
